File: matrix.kicad_sch (KiCad schematic)
At the start: 130 parts, among them SW1 SW_Push, SW10 SW_Push, SW11 SW_Push, SW12 SW_Push, SW13 SW_Push, SW14 SW_Push, SW15 SW_Push, SW16 SW_Push, SW17 SW_Push, SW18 SW_Push, SW19 SW_Push, SW2 SW_Push, SW20 SW_Push, SW21 SW_Push, SW22 SW_Push, SW23 SW_Push, SW24 SW_Push, SW25 SW_Push, SW26 SW_Push, SW27 SW_Push, SW28 SW_Push, SW29 SW_Push, SW3 SW_Push, SW30 SW_Push, SW31 SW_Push, SW32 SW_Push, SW33 SW_Push, SW34 SW_Push, SW35 SW_Push, SW36 SW_Push, SW37 SW_Push, SW38 SW_Push, SW39 SW_Push, SW4 SW_Push, SW40 SW_Push, SW41 SW_Push, SW42 SW_Push, SW43 SW_Push, SW44 SW_Push, SW45 SW_Push, SW46 SW_Push, SW47 SW_Push, SW48 SW_Push, SW49 SW_Push, SW5 SW_Push, SW50 SW_Push, SW51 SW_Push, SW52 SW_Push, SW53 SW_Push, SW54 SW_Push, SW55 SW_Push, SW56 SW_Push, SW57 SW_Push, SW58 SW_Push, SW59 SW_Push, SW6 SW_Push, SW60 SW_Push, SW61 SW_Push, SW62 SW_Push, SW63 SW_Push, SW64 SW_Push, SW65 SW_Push, SW7 SW_Push, SW8 SW_Push, SW9 SW_Push

Commit message: Annotations/ERC Run
Parts:
- SW1: value SW_Push -> `
- SW10: value SW_Push -> 9
- SW11: value SW_Push -> 0
- SW12: value SW_Push -> -
- SW13: value SW_Push -> =
- SW14: value SW_Push -> BKSPC
- SW15: value SW_Push -> DEL
- SW16: value SW_Push -> TAB
- SW17: value SW_Push -> Q
- SW18: value SW_Push -> W
- SW19: value SW_Push -> E
- SW2: value SW_Push -> 1
- SW20: value SW_Push -> R
- SW21: value SW_Push -> T
- SW22: value SW_Push -> Y
- SW23: value SW_Push -> U
- SW24: value SW_Push -> I
- SW25: value SW_Push -> O
- SW26: value SW_Push -> P
- SW27: value SW_Push -> [{
- SW28: value SW_Push -> ]}
- SW29: value SW_Push -> \|
- SW3: value SW_Push -> 2
- SW30: value SW_Push -> HOME
- SW31: value SW_Push -> CAPS
- SW32: value SW_Push -> A
- SW33: value SW_Push -> S
- SW34: value SW_Push -> D
- SW35: value SW_Push -> F
- SW36: value SW_Push -> G
- SW37: value SW_Push -> H
- SW38: value SW_Push -> J
- SW39: value SW_Push -> K
- SW4: value SW_Push -> 3
- SW40: value SW_Push -> L
- SW41: value SW_Push -> ;:
- SW42: value SW_Push -> '"
- SW43: value SW_Push -> ENTER
- SW44: value SW_Push -> LSHIFT
- SW45: value SW_Push -> Z
- SW46: value SW_Push -> X
- SW47: value SW_Push -> C
- SW48: value SW_Push -> V
- SW49: value SW_Push -> B
- SW5: value SW_Push -> 4
- SW50: value SW_Push -> N
- SW51: value SW_Push -> M
- SW52: value SW_Push -> ,<
- SW53: value SW_Push -> .>
- SW54: value SW_Push -> /?
- SW55: value SW_Push -> RSHIFT
- SW56: value SW_Push -> UP
- SW57: value SW_Push -> LCTRL
- SW58: value SW_Push -> LWIN
- SW59: value SW_Push -> LALT
- SW6: value SW_Push -> 5
- SW60: value SW_Push -> SPACE
- SW61: value SW_Push -> RALT
- SW62: value SW_Push -> FN
- SW63: value SW_Push -> LEFT
- SW64: value SW_Push -> DOWN
- SW65: value SW_Push -> RIGHT
- SW7: value SW_Push -> 6
- SW8: value SW_Push -> 7
- SW9: value SW_Push -> 8

Commit message: Footprints Assigned
Parts:
- D1, D10, D11, D12, D13, D14, D15, D16, D17, D18, D19, D2, D20, D21, D22, D23, D24, D25, D26, D27, D28, D29, D3, D30, D31, D32, D33, D34, D35, D36, D37, D38, D39, D4, D40, D41, D42, D43, D44, D45, D46, D47, D48, D49, D5, D50, D51, D52, D53, D54, D55, D56, D57, D58, D59, D6, D60, D61, D62, D63, D64, D65, D7, D8, D9: footprint (none) -> Diode_SMD:D_SOD-123
- SW1, SW10, SW11, SW12, SW13, SW15, SW17, SW18, SW19, SW2, SW20, SW21, SW22, SW23, SW24, SW25, SW26, SW27, SW28, SW3, SW30, SW32, SW33, SW34, SW35, SW36, SW37, SW38, SW39, SW4, SW40, SW41, SW42, SW45, SW46, SW47, SW48, SW49, SW5, SW50, SW51, SW52, SW53, SW54, SW56, SW6, SW63, SW64, SW65, SW7, SW8, SW9: footprint (none) -> MX_Only:MXOnly-1U
- SW14: footprint (none) -> MX_Only:MXOnly-2U
- SW16, SW29: footprint (none) -> MX_Only:MXOnly-1.5U
- SW31, SW55: footprint (none) -> MX_Only:MXOnly-1.75U
- SW43, SW44: footprint (none) -> MX_Only:MXOnly-2.25U
- SW57, SW58, SW59, SW61, SW62: footprint (none) -> MX_Only:MXOnly-1.25U
- SW60: footprint (none) -> MX_Only:MXOnly-6.25U
