File: KeyboardM.kicad_pcb (KiCad board)
At the start: 2 copper layers, 151 parts, among them J1 AVR-ISP-6, SW1 `, SW10 9, SW11 0, SW12 -, SW13 =, SW14 BKSPC, SW15 DEL, SW16 TAB, SW17 Q, SW18 W, SW19 E, SW2 1, SW20 R, SW21 T, SW22 Y, SW23 U, SW24 I, SW25 O, SW26 P, SW27 [{, SW28 ]}, SW29 \|, SW3 2, SW30 HOME, SW31 CAPS, SW32 A, SW33 S, SW34 D, SW35 F, SW36 G, SW37 H, SW38 J, SW39 K, SW4 3, SW40 L, SW41 ;:, SW42 '", SW43 ENTER, SW44 LSHIFT, SW45 Z, SW46 X, SW47 C, SW48 V, SW49 B, SW5 4, SW50 N, SW51 M, SW52 ,<, SW53 .>, SW54 /?, SW55 RSHIFT, SW56 UP, SW57 LCTRL, SW58 LWIN, SW59 LALT, SW6 5, SW60 SPACE, SW61 RALT, SW62 FN, SW63 LEFT, SW64 DOWN, SW65 RIGHT, SW66 SW_Push_Reset, SW7 6, SW8 7, SW9 8, U1 ATmega32U4-A, U2 PRTR5V0U2X, Y1 Crystal_GND24_Small

Commit message: Part 2 Complete
Parts:
- removed SW66: SW_Push_Reset, Button_Switch_SMD:SW_SPST_SKQG_WithStem
- added RSW1: SW_PUSH_RESET, Button_Switch_SMD:SW_SPST_SKQG_WithStem, B.Cu at (235.0, 134.0)
- C1, C2, C3, C4, C5, C6, C7, C8, D1, D10, D11, D12, D13, D14, D15, D16, D17, D18, D19, D2, D20, D21, D22, D23, D24, D25, D26, D27, D28, D29, D3, D30, D31, D32, D33, D34, D35, D36, D37, D38, D39, D4, D40, D41, D42, D43, D44, D45, D46, D47, D48, D49, D5, D50, D51, D52, D53, D54, D55, D56, D57, D58, D59, D6, D60, D61, D62, D63, D64, D65, D7, D8, D9, F1, J1, U1, U2, USB1, Y1: moved to B.Cu
- R1, R2, R3, R4, R5, R6: footprint MX_Only:MXOnly-1U -> Resistor_SMD:R_0805_2012Metric_Pad1.20x1.40mm_HandSolder; moved to B.Cu
- moved D15 311.8 mm to (356.7, 61.9), turned to 90 degrees
- moved D30 285.8 mm to (356.7, 80.8), turned to 90 degrees
- moved D56 277.2 mm to (337.7, 119.1), turned to 90 degrees
- moved D64 267.9 mm to (337.7, 138.0), turned to 90 degrees
- moved D29 264.0 mm to (332.9, 80.9), turned to 90 degrees
- moved D43 259.6 mm to (325.8, 99.9), turned to 90 degrees
- moved D13 257.2 mm to (299.6, 61.9), turned to 90 degrees
- moved D65 255.3 mm to (356.7, 138.0), turned to 90 degrees
- moved SW29 246.8 mm to (327.0, 76.2)
- moved D63 243.7 mm to (318.6, 138.1), turned to 90 degrees
- moved D12 235.2 mm to (280.5, 61.9), turned to 90 degrees
- moved SW55 223.1 mm to (305.6, 114.3)
- moved SW30 219.5 mm to (350.8, 76.2)
- moved D27 219.1 mm to (290.1, 80.9), turned to 90 degrees
- moved D55 217.1 mm to (311.5, 119.0), turned to 90 degrees
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Other:
- board outline added: 304.8 x 99.2 mm

Commit message: Wiring
Parts:
- moved D8 11.8 mm to (192.6, 61.8)
- moved F1 7.27 mm to (204.4, 61.7)
- moved R6 2.09 mm to (204.0, 54.8), turned to 0 degrees
- moved U2 1.70 mm to (208.0, 60.3)
- moved R5 0.53 mm to (210.4, 54.8)
- turned C2 to 0 degrees
- turned Y1 to 90 degrees
Connections:
- R3 pad 1: Net-(R3-Pad1) -> DN
- R4 pad 1: Net-(R4-Pad1) -> DP
- SW60 pad 1: col6 -> col5
- SW61 pad 1: col10 -> col9
- U2 pad 2: Net-(R4-Pad1) -> DP
- U2 pad 3: Net-(R3-Pad1) -> DN
- USB1 pad 5: Net-(R4-Pad1) -> DN
- USB1 pad 6: Net-(R4-Pad1) -> DP
- USB1 pad 7: Net-(R3-Pad1) -> DN
- USB1 pad 8: Net-(R4-Pad1) -> DP
Routing:
- net row1: track 0.00 -> 279.2 mm
- net row0: track 0.00 -> 276.0 mm
- net row3: track 0.00 -> 248.5 mm
- net row2: track 0.00 -> 245.3 mm
- net row4: track 0.00 -> 148.4 mm
- net col1: track 0.00 -> 93.4 mm
- net col2: track 0.00 -> 91.5 mm
- net col11: track 0.00 -> 89.2 mm
- net col9: track 0.00 -> 87.6 mm
- net col5: track 0.00 -> 87.0 mm
- net col13: track 0.00 -> 86.1 mm
- net col0: track 0.00 -> 85.1 mm
- net col12: track 0.00 -> 84.1 mm
- net DN: track 0.00 -> 77.3 mm
- net DP: track 0.00 -> 77.2 mm
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
Commit message: Routing Complete
Parts:
- SW1: value ` -> `~
- SW12: value - -> -_
- SW13: value = -> =+
- SW60: footprint MX_Only:MXOnly-6.25U -> MX_Only:MXOnly-6.25U-ReversedStabilizers
- moved J1 75.3 mm to (242.2, 127.0), turned to 0 degrees
- moved C8 18.9 mm to (232.0, 127.2)
- moved RSW1 17.1 mm to (250.3, 126.2), turned to 0 degrees
- moved C3 10.6 mm to (218.2, 117.5)
- moved R1 7.44 mm to (234.9, 134.1)
- moved R3 6.02 mm to (211.2, 113.7)
- moved R4 6.02 mm to (213.5, 113.7)
- moved C6 4.62 mm to (200.3, 123.6)
- moved R2 3.59 mm to (203.1, 139.3)
- moved D50 2.46 mm to (206.8, 118.2)
- moved Y1 1.23 mm to (220.7, 132.9)
- moved C1 1.23 mm to (226.3, 134.5)
- moved C2 1.23 mm to (226.3, 131.3)
- moved R6 0.49 mm to (204.0, 55.3), turned to 180 degrees
- moved R5 0.33 mm to (210.4, 55.1)
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Connections:
- U1 pad 1: row0 -> row3
- U1 pad 36: col6 -> row4
- U1 pad 38: row1 -> col6
- U1 pad 39: row4 -> row0
- U1 pad 40: row3 -> row1
Routing:
- net GND: track 13.4 -> 317.7 mm, vias 0 -> 9
- net row0: track 276.0 -> 492.5 mm, vias 0 -> 4
- net +5V: track 0.00 -> 196.6 mm, vias 0 -> 6
- net row1: track 279.2 -> 463.8 mm, vias 0 -> 4
- net row2: track 245.3 -> 409.1 mm, vias 0 -> 4
- net row4: track 148.4 -> 311.9 mm, vias 0 -> 2
- net col0: track 85.1 -> 246.0 mm, vias 0 -> 1
- net col14: track 76.2 -> 224.0 mm, vias 0 -> 1
- net col1: track 93.4 -> 222.8 mm, vias 0 -> 1
- net col13: track 86.1 -> 213.5 mm, vias 0 -> 1
- net col12: track 84.1 -> 191.5 mm, vias 0 -> 1
- net col2: track 91.5 -> 195.3 mm, vias 0 -> 1
- net col3: track 67.0 -> 150.8 mm, vias 0 -> 1
- net col8: track 67.0 -> 146.7 mm, vias 0 -> 1
- net col10: track 67.0 -> 146.6 mm, vias 0 -> 1
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- added copper zone on B.Cu, net (none)
- added copper zone on F.Cu, net (none)

Commit message: v1.0.0
Parts:
- added FB1: 60@100MHz, Inductor_SMD:L_0805_2012Metric_Pad1.15x1.40mm_HandSolder, B.Cu at (216.5, 49.8)
- moved R5 0.46 mm to (210.4, 55.6), turned to -90 degrees
Connections:
- USB1 pad 13: GND -> Earth
Routing:
- net GND: track 317.7 -> 338.6 mm, vias 9 -> 82
- net Earth: track 0.00 -> 15.6 mm, vias 0 -> 5
- net VCC: track 20.1 -> 25.4 mm
- net col10: track 146.6 -> 144.5 mm
- net row3: track 276.2 -> 275.2 mm
- net +5V: track 196.6 -> 197.3 mm
- added copper zone on B.Cu, net Earth
- added copper zone on B.Cu, net GND
- added copper zone on F.Cu, net GND
