File: KeyboardM.kicad_pcb (KiCad board)
At the start: 2 copper layers, 304.8 x 99.2 mm, 152 parts, among them J1 AVR-ISP-6, SW1 `~, SW10 9, SW11 0, SW12 -_, SW13 =+, SW14 BKSPC, SW15 DEL, SW16 TAB, SW17 Q, SW18 W, SW19 E, SW2 1, SW20 R, SW21 T, SW22 Y, SW23 U, SW24 I, SW25 O, SW26 P, SW27 [{, SW28 ]}, SW29 \|, SW3 2, SW30 HOME, SW31 CAPS, SW32 A, SW33 S, SW34 D, SW35 F, SW36 G, SW37 H, SW38 J, SW39 K, SW4 3, SW40 L, SW41 ;:, SW42 '", SW43 ENTER, SW44 LSHIFT, SW45 Z, SW46 X, SW47 C, SW48 V, SW49 B, SW5 4, SW50 N, SW51 M, SW52 ,<, SW53 .>, SW54 /?, SW55 RSHIFT, SW56 UP, SW57 LCTRL, SW58 LWIN, SW59 LALT, SW6 5, SW60 SPACE, SW61 RALT, SW62 FN, SW63 LEFT, SW64 DOWN, SW65 RIGHT, SW7 6, SW8 7, SW9 8, U1 ATmega32U4-A, U2 PRTR5V0U2X, Y1 Crystal_GND24_Small

Commit message: v1.0.1
Parts:
- moved C8 32.3 mm to (199.7, 126.2)
Routing:
- net GND: track 338.6 -> 331.2 mm, vias 82 -> 81
- net RESET: track 66.6 -> 63.7 mm
- net SCK: track 36.4 -> 34.1 mm
- net MOSI: track 37.9 -> 35.9 mm
- net +5V: track 197.3 -> 195.6 mm
- net MISO: track 33.0 -> 31.6 mm
